Commit message: a lot of change

File: mobile_manipulator/mobile_manipulator_description/urdf/khi_rs/rs005l_macro.xacro (robot description, xacro)
@@ -234,69 +234,87 @@
       <xacro:default_inertial mass="${j6_mass}"/>
     </link>
-	    <link name="camera_link">
-		    <visual>
-			<origin xyz="-0.03 0 0" rpy="-1.57 0 -1.57"/>
-			<geometry>
-			    <mesh filename="package://mobile_manipulator_description/meshes/camera.stl" scale="0.001 0.001 0.001"/>
-			</geometry>
-		    </visual>
-	    </link>
-	    <joint name="camera_joint" type="fixed">
-			<origin xyz="0.0 0.0 0.03" rpy="-1.570796 -1.570796 0"/>
-			<parent link="link6"/>
-			<child link="camera_link"/>
-	    </joint>
-	    <joint name="camera_rgb_joint" type="fixed">
-			<origin xyz="0 0 0" rpy="-1.570796 0 -1.570796"/>
-			<parent link="camera_link"/>
-			<child link="camera_rgb_frame"/>
-	    </joint>
-	    <link name="camera_rgb_frame"/>
-	    <joint name="camera_rgb_optic_joint" type="fixed">
-			<origin xyz="0 0 0" rpy="0 0 0"/>
-			<parent link="camera_rgb_frame"/>
-			<child link="camera_rgb_optic_frame"/>
-	    </joint>
-   	 <link name="camera_rgb_optic_frame"/>
-	  <gazebo reference="camera_link">
-	    <sensor type="depth" name="Realsense_Camera_Depth">
-	      <always_on>true</always_on>
-	      <update_rate>10.0</update_rate>
-			<camera>
-				<horizontal_fov>1.3962634</horizontal_fov>
-				<image>
-					<width>640</width>
-					<height>480</height>
-					<format>R8G8B8</format>
-				</image>
-				<clip>
-					<near>0.01</near>
-					<far>5</far>
-				</clip>
-			</camera>
-		<plugin name="depth_camera_plugin" filename="libgazebo_ros_openni_kinect.so">
-			  <alwaysOn>true</alwaysOn>
-			  <updateRate>10.0</updateRate>
-			  <cameraName>camera</cameraName>
-			  <imageTopicName>image_raw</imageTopicName>
-			  <cameraInfoTopicName>camera_info</cameraInfoTopicName>
-			  <depthImageTopicName>depth_image_raw</depthImageTopicName>
-			  <depthImageCameraInfoTopicName>depth_camera_info</depthImageCameraInfoTopicName>
-			  <pointCloudTopicName>points</pointCloudTopicName>
-			  <frameName>camera_rgb_optic_frame</frameName>
-			  <pointCloudCutoff>0.0</pointCloudCutoff>
-			  <distortionK1>0.00000001</distortionK1>
-			  <distortionK2>0.00000001</distortionK2>
-			  <distortionK3>0.00000001</distortionK3>
-			  <distortionT1>0.00000001</distortionT1>
-			  <distortionT2>0.00000001</distortionT2>
-			  <CxPrime>0</CxPrime>
-			  <Cx>0</Cx>
-			  <Cy>0</Cy>
-			  <focalLength>0</focalLength>
-			  <hackBaseline>0</hackBaseline>
-		</plugin>
-	    </sensor>
-	  </gazebo>
+    <!-- Link 6 -->
+    <joint name="${prefix}joint7" type="fixed">
+      <axis xyz="0 0 1" rpy="0 0 0" />
+      <origin xyz="0.04 -0.035 0.22" rpy="1.570796 -1.570796 0" />
+      <parent link="${prefix}link6"/>
+      <child link="${prefix}link7"/>
+    </joint>
+        <link name="${prefix}link7">
+      <visual>
+        <geometry>
+          <mesh filename="package://mobile_manipulator_description/meshes/khi_rs/Montaj.stl" scale="0.001 0.001 0.001"/>
+        </geometry>
+        <material name="Black"/>
+        <origin xyz="0 0 0" rpy="0 -1.570796 1.570796"/>
+      </visual>
+      <collision>
+        <geometry>
+          <mesh filename="package://mobile_manipulator_description/meshes/khi_rs/Montaj.stl" scale="0.001 0.001 0.001"/>
+        </geometry>
+        <material name="Black"/>
+        <origin xyz="0 0 0" rpy="0 -1.570796 1.570796"/>
+      </collision>
+      <xacro:default_inertial mass="0.2"/>
+    </link>
+    <link name="camera_link"/>
+    <joint name="camera_joint" type="fixed">
+       <origin xyz="-0.04 0.0525 -0.021" rpy="0 0 0"/>
+       <parent link="${prefix}link7"/>
+       <child link="camera_link"/>
+    </joint>
+    <joint name="camera_rgb_joint" type="fixed">
+       <origin xyz="0 0 0" rpy="0 0 0"/>
+       <parent link="camera_link"/>
+       <child link="camera_rgb_frame"/>
+    </joint>
+    <link name="camera_rgb_frame"/>
+    <joint name="camera_rgb_optic_joint" type="fixed">
+       <origin xyz="0 0 0" rpy="0 0 0"/>
+       <parent link="camera_rgb_frame"/>
+       <child link="camera_rgb_optic_frame"/>
+    </joint>
+    <link name="camera_rgb_optic_frame"/>
+    <gazebo reference="camera_link">
+      <sensor type="depth" name="Realsense_Camera_Depth">
+      <always_on>true</always_on>
+      <update_rate>10.0</update_rate>
+      <camera>
+        <horizontal_fov>1.22</horizontal_fov>
+        <image>
+          <width>512</width>
+          <height>424</height>
+          <format>R8G8B8</format>
+        </image>
+        <clip>
+          <near>0.01</near>
+          <far>16</far>
+        </clip>
+      </camera>
+      <plugin name="depth_camera_plugin" filename="libgazebo_ros_openni_kinect.so">
+        <visualize>true</visualize>
+        <alwaysOn>true</alwaysOn>
+        <updateRate>10.0</updateRate>
+        <cameraName>camera</cameraName>
+        <imageTopicName>image_raw</imageTopicName>
+        <cameraInfoTopicName>camera_info</cameraInfoTopicName>
+        <depthImageTopicName>depth_image_raw</depthImageTopicName>
+        <depthImageCameraInfoTopicName>depth_camera_info</depthImageCameraInfoTopicName>
+        <pointCloudTopicName>points</pointCloudTopicName>
+        <frameName>camera_rgb_optic_frame</frameName>
+        <pointCloudCutoff>0.0</pointCloudCutoff>
+        <distortionK1>0.00000001</distortionK1>
+        <distortionK2>0.00000001</distortionK2>
+        <distortionK3>0.00000001</distortionK3>
+        <distortionT1>0.00000001</distortionT1>
+        <distortionT2>0.00000001</distortionT2>
+        <CxPrime>0</CxPrime>
+        <Cx>0</Cx>
+        <Cy>0</Cy>
+        <focalLength>0</focalLength>
+        <hackBaseline>0</hackBaseline>
+      </plugin>
+      </sensor>
+    </gazebo>
   </xacro:macro>
 </robot>

Commit message: Updated description

File: mobile_manipulator/mobile_manipulator_description/urdf/khi_rs/rs005l_macro.xacro (robot description, xacro)
@@ -234,8 +234,8 @@
       <xacro:default_inertial mass="${j6_mass}"/>
     </link>
-    <!-- Link 6 -->
+    <!-- Link 7 -->
     <joint name="${prefix}joint7" type="fixed">
       <axis xyz="0 0 1" rpy="0 0 0" />
-      <origin xyz="0.04 -0.035 0.22" rpy="1.570796 -1.570796 0" />
+      <origin xyz="0 0 0" rpy="0 0 -1.96" />
       <parent link="${prefix}link6"/>
       <child link="${prefix}link7"/>
@@ -247,5 +247,5 @@
         </geometry>
         <material name="Black"/>
-        <origin xyz="0 0 0" rpy="0 -1.570796 1.570796"/>
+        <origin xyz="-0.035 -0.04 0.2175" rpy="1.570796 3.1415 0"/>
       </visual>
       <collision>
@@ -254,11 +254,12 @@
         </geometry>
         <material name="Black"/>
-        <origin xyz="0 0 0" rpy="0 -1.570796 1.570796"/>
-      </collision>
-      <xacro:default_inertial mass="0.2"/>
-    </link>
+        <origin xyz="-0.035 -0.04 0.2175" rpy="1.570796 3.1415 0"/>
+      </collision>
+      <xacro:default_inertial mass="0.1"/>
+    </link>
+<!--
     <link name="camera_link"/>
     <joint name="camera_joint" type="fixed">
-       <origin xyz="-0.04 0.0525 -0.021" rpy="0 0 0"/>
+       <origin xyz="0.0145 0.0125 0.185" rpy="0 -1.570796 1.570796"/>
        <parent link="${prefix}link7"/>
        <child link="camera_link"/>
@@ -292,6 +293,6 @@
         </clip>
       </camera>
+      <visualize>True</visualize>
       <plugin name="depth_camera_plugin" filename="libgazebo_ros_openni_kinect.so">
-        <visualize>true</visualize>
         <alwaysOn>true</alwaysOn>
         <updateRate>10.0</updateRate>
@@ -316,5 +317,5 @@
       </plugin>
       </sensor>
-    </gazebo>
+    </gazebo>-->
   </xacro:macro>
 </robot>

File: mobile_manipulator/mobile_manipulator_description/urdf/ota/ota_base.xacro (robot description, xacro)
@@ -11,7 +11,7 @@
       </visual>
       <collision>
-        <origin xyz="0 0 -0.0" rpy=" 0 0 0"/>
+        <origin xyz="0 0 0.015" rpy=" 0 0 0"/>
         <geometry>
-          <box size="1.02605 0.728 0.25"/>
+          <box size="1.02605 0.728 0.3"/>
         </geometry>
       </collision>
@@ -45,4 +45,5 @@
     <origin rpy="0 0 0" xyz="0.001 -0.26 0.212"/>
   </joint>
+<!--
 	    <link name="camera1_link">
 		    <visual>
@@ -176,4 +177,5 @@
 	    </sensor>
 	  </gazebo>
+	-->
   </xacro:macro>
 </robot>

File: mobile_manipulator/mobile_manipulator_description/urdf/ota/ota_plugin.xacro (robot description, xacro)
@@ -25,6 +25,6 @@
       <plugin name="differential_drive_controller" filename="libgazebo_ros_diff_drive.so">
         <robotNamespace>/</robotNamespace>
-        <publishOdomTF>true</publishOdomTF>
-        <publishWheelJointState>true</publishWheelJointState>
+        <publishOdomTF>false</publishOdomTF>
+        <publishWheelJointState>false</publishWheelJointState>
         <alwaysOn>true</alwaysOn>
         <leftJoint>wheel_right_base</leftJoint>
@@ -34,11 +34,11 @@
         <wheelTorque>20</wheelTorque>
         <wheelAcceleration>1.8</wheelAcceleration>
-        <commandTopic>cmd_vel</commandTopic>
-        <odometryTopic>odom</odometryTopic>
-        <odometryFrame>odom</odometryFrame>
+        <commandTopic>sim_cmd_vel</commandTopic>
+        <odometryTopic>sim_odom</odometryTopic>
+        <odometryFrame>sim_odom</odometryFrame>
         <odometrySource>world</odometrySource>
         <robotBaseFrame>${base_link}</robotBaseFrame>
 	      <legacyMode>true</legacyMode>
-	      <publishTf>true</publishTf>
+	      <publishTf>false</publishTf>
         <updateRate>50.0</updateRate>
       </plugin>
