Commit message: Updated config

File: mobile_manipulator/mobile_manipulator_moveit_config/config/gazebo_robot (copy).urdf (robot description, URDF)
Before this commit: robot robot, 30 links, 29 joints
Links:
- link link7: mass 0.1 -> 0.2
Joints:
- joint camera_joint: origin xyz=0.0145 0.0125 0.185 rpy=0 -1.570796 1.570796 -> xyz=-0.04 0.0525 -0.021 rpy=0 0 0
- joint joint7: origin xyz=0 0 0 rpy=0 0 0 -> xyz=0.04 -0.035 0.22 rpy=1.570796 -1.570796 0
